File: mosaic-x3.kicad_pcb (KiCad board)
At the start: 2 copper layers, 21 x 130 mm, 33 parts, among them J1 Conn_01x02, J2 USB_C_Receptacle_USB2.0_14P, J3 LED_STRIP_HEAD, J4 PWR_INJ_1, J5 PWR_INJ_2, J6 PWR_INJ_3, Q1 P-MOSFET, SW1 SW_SPST, SW2 RESET, SW3 BOOT, U1 AMS1117-3.3, U2 ESP32-S3-WROOM-1, U3 74AHCT125

Commit message: bump updates
Parts:
- removed J6: PWR_INJ_3, Connector_JST:JST_XH_S2B-XH-A_1x02_P2.50mm_Horizontal
- added REF**: MountingHole_2.7mm_M2.5, MountingHole:MountingHole_2.7mm_M2.5, F.Cu at (105.0, 173.3)
- added REF**: MountingHole_2.7mm_M2.5, MountingHole:MountingHole_2.7mm_M2.5, F.Cu at (104.4, 101.5)
- F1: footprint Fuse:Fuse_1812_4532Metric -> Fuse:Fuse_2920_7451Metric_Pad2.10x5.45mm_HandSolder
- moved J1 13.3 mm to (105.3, 115.8), turned to 180 degrees
- moved F1 12.5 mm to (103.3, 123.6)
- moved J5 12.1 mm to (90.3, 172.6)
- moved J3 11.8 mm to (90.4, 153.5)
- moved J4 11.7 mm to (90.4, 163.1)
- moved R5 11.6 mm to (90.8, 144.3), turned to 180 degrees
- moved C1 11.2 mm to (103.6, 139.9)
- moved Q1 10.6 mm to (104.1, 131.7), turned to 90 degrees
- moved C3 10.5 mm to (98.9, 134.7), turned to -90 degrees
- moved C2 10.0 mm to (98.9, 130.6), turned to -90 degrees
- moved D1 8.32 mm to (96.3, 119.0), turned to -90 degrees
- moved R7 7.47 mm to (96.2, 144.0), turned to 0 degrees
- moved R9 7.05 mm to (96.2, 139.3), turned to 0 degrees
- moved R8 6.44 mm to (96.2, 141.6), turned to 0 degrees
- moved R6 5.95 mm to (96.2, 125.9), turned to -90 degrees
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Routing:
- net Net-(Q1-G): track 11.7 -> 25.4 mm
- net Net-(R5-Pad2): track 50.2 -> 61.7 mm
- net Net-(D1-K): track 15.4 -> 25.8 mm
- net +3V3: track 106.0 -> 112.5 mm, vias 3 -> 5
- net STATUS_R: track 91.3 -> 85.8 mm
- net STATUS_G: track 89.3 -> 84.1 mm
- net GND: track 19.0 -> 23.8 mm
- net STATUS_B: track 86.8 -> 82.5 mm
- net Net-(D2-BA): track 7.10 -> 4.64 mm
- net Net-(D2-GA): track 7.23 -> 4.95 mm
- net USB_DM: track 23.6 -> 25.6 mm
- net +5V: track 130.5 -> 128.5 mm, vias 0 -> 4
- net USB_VBUS: track 7.62 -> 9.14 mm
- net Net-(J1-Pin_1): track 9.44 -> 8.11 mm
- net Net-(D2-RA): track 5.32 -> 6.12 mm
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Other:
- board size 21 x 130 mm -> 21 x 128 mm
