File: mosaic-x3.kicad_sch (KiCad schematic)
At the start: 33 parts, among them J1 Conn_01x02, J2 USB_C_Receptacle_USB2.0_14P, J3 LED_STRIP_HEAD, J4 PWR_INJ_1, J5 PWR_INJ_2, J6 PWR_INJ_3, Q1 P-MOSFET, SW1 SW_SPST, SW2 RESET, SW3 BOOT, U1 AMS1117-3.3, U2 ESP32-S3-WROOM-1, U3 74AHCT125

Commit message: bump updates
Parts:
- removed J6: PWR_INJ_3, Connector_JST:JST_XH_S2B-XH-A_1x02_P2.50mm_Horizontal, symbol Connector_Generic:Conn_01x02
- F1: footprint Fuse:Fuse_1812_4532Metric -> Fuse:Fuse_2920_7451Metric_Pad2.10x5.45mm_HandSolder
Other:
- moved on the sheet: J3, J4, J5

Commit message: fixed project
Other:
- note added: "Mosaic-X3 schematics (v1): 12 weeks = 84 LEDs (12x7) lights: 5V WS2812B 60/m strip Firmware NUM_LEDS = 84"
- note added: "connect a regulated 5V DC supply to this terminal for power"
- note removed: "Mosaic-X3 schematics (v1): 26 weeks (6mo) = 182 LEDs lights: 5V WS2812B 60/m strip Firmware NUM_LEDS = 182"
- note removed: "we will connect panel mount barrel jack to this connector for power"
Changed lines of the file:
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@@
 		)
 	)
-	(text "we will connect panel \nmount barrel jack to \nthis connector for power"
+	(text "connect a regulated 5V \nDC supply to this \nterminal for power"
 		(exclude_from_sim no)
 		(at 159.004 37.338 0)
@@
 		)
 	)
-	(text "Mosaic-X3 schematics (v1):\n26 weeks (6mo) = 182 LEDs\nlights: 5V WS2812B 60/m strip\nFirmware NUM_LEDS = 182"
+	(text "Mosaic-X3 schematics (v1):\n12 weeks = 84 LEDs (12x7)\nlights: 5V WS2812B 60/m strip\nFirmware NUM_LEDS = 84"
 		(exclude_from_sim no)
 		(at 177.292 159.258 0)
